Commit message: Add fused localization and map management workflows

File: src/Go2_URDF/GO2_URDF/urdf/go2_description.urdf (robot description, URDF)
Before this commit: robot go2_description, 32 links, 31 joints
Links:
- added link base_footprint
Joints:
- added joint base_footprint_to_base_link: type fixed, parent base_footprint, child base_link, origin xyz=0 0 0.32 rpy=0 0 0
